File: hardware/KungFuFlash.sch (KiCad schematic (older format))
At the start: 38 parts, among them J1 USB Power, J2 USB_B_Micro, J4 SWD, Q1 BC817, SW1 Reset, SW2 Menu, SW3 Special, U1 C64-Exp-Port, U2 AMS1117-3.3, U3 STM32F405RGTx, Y1 8MHz

Commit message: Change to LQFP-100, replace resitor network, add DMA
Parts:
- removed RN1, RN2: 100R, Resistor_SMD:R_Array_Convex_4x0603, symbol Device:R_Pack04
- removed U3: STM32F405RGTx, Package_QFP:LQFP-64_10x10mm_P0.5mm, symbol MCU_ST_STM32F4:STM32F405RGTx
- added R10, R11, R12, R13, R14, R15, R7, R8, R9: 100R, Resistor_SMD:R_0603_1608Metric_Pad0.98x0.95mm_HandSolder, symbol Device:R
- added U3: STM32F407VETx, Package_QFP:LQFP-100_14x14mm_P0.5mm, symbol MCU_ST_STM32F4:STM32F407VETx
- J2: symbol Connector:USB_B_Micro -> KungFuFlash-rescue:USB_B_Micro-Connector-KungFuFlash-rescue
Connections:
- net labels added: CDMA, DMA
- wire segments 218 -> 232
- no-connect marks 4 -> 3
Other:
- moved on the sheet: C16, C17, J4, Q1, R3, R4, R5, R6, SW2, SW3
